File: ExtraCore.brd (EAGLE design)
At the start: 19.8 x 22.4 mm, 19 parts, among them Y1 RESONATORSMD

Commit message: Traces and lettering for v1.5
Routing:
- net GND: track 0.00 -> 52.7 mm, vias 0 -> 2
- net VCC: track 0.00 -> 50.3 mm, vias 0 -> 1
- net RESET: track 0.00 -> 27.3 mm, vias 0 -> 2
- net RAW: track 0.00 -> 25.9 mm
- net TX: track 0.00 -> 19.9 mm, vias 0 -> 1
- net A6: track 0.00 -> 16.9 mm, vias 0 -> 1
- net RX: track 0.00 -> 16.9 mm, vias 0 -> 1
- net A7: track 0.00 -> 15.0 mm
- net AREF: track 0.00 -> 12.0 mm
- net A5: track 0.00 -> 11.7 mm
- net SCK: track 0.00 -> 11.4 mm
- net DTR: track 0.00 -> 10.6 mm
- net D4: track 0.00 -> 10.5 mm
- net D6: track 0.00 -> 10.4 mm
- net A4: track 0.00 -> 9.92 mm
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Other:
- board text added: "20121105"
- board text added: "ExtraCore v1.5"
- board text added: "by: Dustin Andrews"
- board text removed: "0.78" x 0.88""
- board text removed: "20110909"
- board text removed: "Andrews"
- board text removed: "ExtraCore"
- board text removed: "by: Dustin"
