File: ExtraCore.brd (EAGLE design)
At the start: 19.8 x 22.4 mm, 19 parts, among them Y1 RESONATORSMD

Commit message: 20121229 updates. Sent to manf.
Parts:
- LED1: value GREEN -> (none); device ExtraCore:LED1206 -> SparkFun:LED-0805
- moved RG1 5.47 mm to (6.65, 11.5)
- moved C4 5.40 mm to (9.02, 18.1)
- moved C5 5.40 mm to (6.73, 18.2)
- moved LED1 0.13 mm to (14.9, 14.5)
Connections:
- net GND: now also LED1.C; no longer LED1.K
Routing:
- net RESET: track 27.3 -> 48.8 mm
- net RAW: track 25.9 -> 15.8 mm
- net GND: track 52.7 -> 57.4 mm, vias 2 -> 4
- net VCC: track 50.3 -> 46.0 mm, vias 1 -> 3
- net TX: track 19.9 -> 16.7 mm
- net D2: track 8.91 -> 10.0 mm
- net A3: track 8.26 -> 9.17 mm
- net A6: track 16.9 -> 17.5 mm
- net D5: track 8.04 -> 8.59 mm
- net A2: track 6.65 -> 6.44 mm, vias 0 -> 1
- added copper zone on layer 1, net GND
- added copper zone on layer 16, net GND
Other:
- board text added: "20121229"
- board text added: "ExtraCore v2"
- board text removed: "20121105"
- board text removed: "ExtraCore v1.5"
