File: ExtraCore.sch (EAGLE design)
At the start: 19 parts, among them Y1 RESONATORSMD

Commit message: 20121229 updates. Sent to manf.
Parts:
- LED1: value GREEN -> (none); device ExtraCore:LED1206 -> SparkFun:LED0805
Connections:
- net GND: now also LED1.C; no longer LED1.K
Changed lines of the file:
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@@
 <?xml version="1.0" encoding="utf-8"?>
 <!DOCTYPE eagle SYSTEM "eagle.dtd">
-<eagle version="6.2">
+<eagle version="6.3">
 <drawing>
 <settings>
@@
 </variantdefs>
 <classes>
-<class number="0" name="default" width="0" drill="0">
+<class number="0" name="default" width="0.2032" drill="0.2032">
+<clearance class="0" value="0.2032"/>
+</class>
+<class number="1" name="GND" width="0.3048" drill="0.2032">
+<clearance class="1" value="0.2032"/>
+</class>
+<class number="2" name="PWR" width="0.3048" drill="0.2032">
+<clearance class="2" value="0.2032"/>
 </class>
 </classes>
@@
 <part name="RESET" library="SparkFun" deviceset="M01" device="PTH"/>
 <part name="L1" library="SparkFun" deviceset="INDUCTOR" device="0805" value="10uH"/>
-<part name="LED1" library="ExtraCore" deviceset="LED" device="1206" value="GREEN"/>
 <part name="RG1" library="Dustin" deviceset="LDO_VREG_3PIN" device="" value="5v"/>
 <part name="C4" library="SparkFun-Passives" deviceset="CAP" device="0805" value="4.7uf"/>
 <part name="C5" library="SparkFun-Passives" deviceset="CAP" device="0805" value="4.7uf"/>
 <part name="GND5" library="SparkFun" deviceset="GND" device=""/>
+<part name="LED1" library="SparkFun" deviceset="LED" device="0805"/>
 </parts>
 <sheets>
@@
 <instance part="RESET" gate="G$1" x="-60.96" y="43.18"/>
 <instance part="L1" gate="G$1" x="-5.08" y="81.28" rot="R180"/>
-<instance part="LED1" gate="A" x="109.22" y="10.16"/>
 <instance part="RG1" gate="G$1" x="-15.24" y="20.32" rot="R90"/>
 <instance part="C4" gate="G$1" x="0" y="15.24" rot="R90"/>
 <instance part="C5" gate="G$1" x="0" y="25.4" rot="R90"/>
 <instance part="GND5" gate="1" x="10.16" y="10.16"/>
+<instance part="LED1" gate="G$1" x="109.22" y="12.7"/>
 </instances>
 <busses>
 </busses>
 <nets>
-<net name="VCC" class="0">
+<net name="VCC" class="2">
 <segment>
 <wire x1="48.26" y1="99.06" x2="48.26" y2="106.68" width="0.1524" layer="91"/>
@@
 </segment>
 </net>
-<net name="GND" class="0">
+<net name="GND" class="1">
 <segment>
 <wire x1="25.4" y1="60.96" x2="25.4" y2="58.42" width="0.1524" layer="91"/>
@@
 <wire x1="109.22" y1="7.62" x2="109.22" y2="2.54" width="0.1524" layer="91"/>
 <pinref part="GND3" gate="1" pin="GND"/>
-<pinref part="LED1" gate="A" pin="K"/>
+<pinref part="LED1" gate="G$1" pin="C"/>
 </segment>
 <segment>
@@
 <wire x1="109.22" y1="17.78" x2="109.22" y2="15.24" width="0.1524" layer="91"/>
 <pinref part="R2" gate="G$1" pin="1"/>
-<pinref part="LED1" gate="A" pin="A"/>
+<pinref part="LED1" gate="G$1" pin="A"/>
 </segment>
 </net>
@@
 </segment>
 </net>
-<net name="RAW" class="0">
+<net name="RAW" class="2">
 <segment>
 <pinref part="RG1" gate="G$1" pin="IN"/>
